File: pcb/pcb.kicad_pcb (KiCad board)
At the start: 2 copper layers, 88.1 x 61.9 mm, 19 parts, among them U1 Raspberry_Pi_Pico

Commit message: still making the full 72 sized keyboard pcb
Parts:
- added D10: Diode, ScottoKeebs_Components:Diode_DO-35, F.Cu at (208.1, 146.8)
- added D11: Diode, ScottoKeebs_Components:Diode_DO-35, F.Cu at (208.1, 150.4)
- added D12: Diode, ScottoKeebs_Components:Diode_DO-35, F.Cu at (208.1, 153.9)
- added D13: Diode, ScottoKeebs_Components:Diode_DO-35, F.Cu at (208.1, 157.5)
- added D14: Diode, ScottoKeebs_Components:Diode_DO-35, F.Cu at (218.9, 114.9)
- added D15: Diode, ScottoKeebs_Components:Diode_DO-35, F.Cu at (218.9, 118.4)
- added D16: Diode, ScottoKeebs_Components:Diode_DO-35, F.Cu at (218.9, 122.0)
- added D17: Diode, ScottoKeebs_Components:Diode_DO-35, F.Cu at (218.9, 125.5)
- added D18: Diode, ScottoKeebs_Components:Diode_DO-35, F.Cu at (218.9, 129.1)
- added D19: Diode, ScottoKeebs_Components:Diode_DO-35, F.Cu at (218.9, 132.6)
- added D20: Diode, ScottoKeebs_Components:Diode_DO-35, F.Cu at (218.9, 136.2)
- added D21: Diode, ScottoKeebs_Components:Diode_DO-35, F.Cu at (218.9, 139.7)
- added D22: Diode, ScottoKeebs_Components:Diode_DO-35, F.Cu at (218.9, 143.3)
- added D23: Diode, ScottoKeebs_Components:Diode_DO-35, F.Cu at (218.9, 146.8)
- added D24: Diode, ScottoKeebs_Components:Diode_DO-35, F.Cu at (218.9, 150.4)
- added D25: Diode, ScottoKeebs_Components:Diode_DO-35, F.Cu at (218.9, 153.9)
- added D26: Diode, ScottoKeebs_Components:Diode_DO-35, F.Cu at (218.9, 157.5)
- added D27: Diode, ScottoKeebs_Components:Diode_DO-35, F.Cu at (229.6, 114.9)
- added D28: Diode, ScottoKeebs_Components:Diode_DO-35, F.Cu at (229.6, 118.4)
- added D29: Diode, ScottoKeebs_Components:Diode_DO-35, F.Cu at (229.6, 122.0)
- added D30: Diode, ScottoKeebs_Components:Diode_DO-35, F.Cu at (229.6, 125.5)
- added D31: Diode, ScottoKeebs_Components:Diode_DO-35, F.Cu at (229.6, 129.1)
- added D32: Diode, ScottoKeebs_Components:Diode_DO-35, F.Cu at (229.6, 132.6)
- added D33: Diode, ScottoKeebs_Components:Diode_DO-35, F.Cu at (229.6, 136.2)
- added D37: Diode, ScottoKeebs_Components:Diode_DO-35, F.Cu at (229.6, 139.7)
- added D38: Diode, ScottoKeebs_Components:Diode_DO-35, F.Cu at (229.6, 143.3)
- added D39: Diode, ScottoKeebs_Components:Diode_DO-35, F.Cu at (229.6, 146.8)
- added D40: Diode, ScottoKeebs_Components:Diode_DO-35, F.Cu at (229.6, 150.4)
- added D41: Diode, ScottoKeebs_Components:Diode_DO-35, F.Cu at (229.6, 153.9)
- added D42: Diode, ScottoKeebs_Components:Diode_DO-35, F.Cu at (229.6, 157.5)
- added D43: Diode, ScottoKeebs_Components:Diode_DO-35, F.Cu at (240.4, 114.9)
- added D44: Diode, ScottoKeebs_Components:Diode_DO-35, F.Cu at (240.4, 118.4)
- added D45: Diode, ScottoKeebs_Components:Diode_DO-35, F.Cu at (240.4, 122.0)
- added D46: Diode, ScottoKeebs_Components:Diode_DO-35, F.Cu at (240.4, 125.5)
- added D47: Diode, ScottoKeebs_Components:Diode_DO-35, F.Cu at (240.4, 129.1)
- added D48: Diode, ScottoKeebs_Components:Diode_DO-35, F.Cu at (240.4, 132.6)
- added D49: Diode, ScottoKeebs_Components:Diode_DO-35, F.Cu at (240.4, 136.2)
- added D50: Diode, ScottoKeebs_Components:Diode_DO-35, F.Cu at (240.4, 139.7)
- added D51: Diode, ScottoKeebs_Components:Diode_DO-35, F.Cu at (240.4, 143.3)
- added D52: Diode, ScottoKeebs_Components:Diode_DO-35, F.Cu at (240.4, 146.8)
- added D53: Diode, ScottoKeebs_Components:Diode_DO-35, F.Cu at (240.4, 150.4)
- added D54: Diode, ScottoKeebs_Components:Diode_DO-35, F.Cu at (240.4, 153.9)
- added D55: Diode, ScottoKeebs_Components:Diode_DO-35, F.Cu at (240.4, 157.5)
- added D56: Diode, ScottoKeebs_Components:Diode_DO-35, F.Cu at (251.2, 114.9)
- added D57: Diode, ScottoKeebs_Components:Diode_DO-35, F.Cu at (251.2, 118.4)
- added D58: Diode, ScottoKeebs_Components:Diode_DO-35, F.Cu at (251.2, 122.0)
- added D59: Diode, ScottoKeebs_Components:Diode_DO-35, F.Cu at (251.2, 125.5)
- added D61: Diode, ScottoKeebs_Components:Diode_DO-35, F.Cu at (251.2, 129.1)
- added D63: Diode, ScottoKeebs_Components:Diode_DO-35, F.Cu at (251.2, 132.6)
- added D67: Diode, ScottoKeebs_Components:Diode_DO-35, F.Cu at (251.2, 136.2)
- added D71: Diode, ScottoKeebs_Components:Diode_DO-35, F.Cu at (251.2, 139.7)
- added D72: Diode, ScottoKeebs_Components:Diode_DO-35, F.Cu at (251.2, 143.3)
- added S10: 3, ScottoKeebs_MX:MX_PCB_1.00u, F.Cu at (79.2, 54.0)
- added S11: e, ScottoKeebs_MX:MX_PCB_1.00u, F.Cu at (88.7, 73.0)
- added S12: d, ScottoKeebs_MX:MX_PCB_1.00u, F.Cu at (51.5, 114.6)
- added S13: 4, ScottoKeebs_MX:MX_PCB_1.00u, F.Cu at (98.2, 54.0)
- added S14: r, ScottoKeebs_MX:MX_PCB_1.00u, F.Cu at (107.8, 73.0)
- added S15: f, ScottoKeebs_MX:MX_PCB_1.00u, F.Cu at (84.5, 135.0)
- added S16: 5, ScottoKeebs_MX:MX_PCB_1.00u, F.Cu at (117.3, 54.0)
- added S17: t, ScottoKeebs_MX:MX_PCB_1.00u, F.Cu at (73.3, 160.5)
- added S18: g, ScottoKeebs_MX:MX_PCB_1.00u, F.Cu at (84.5, 181.6)
- added S19: 6, ScottoKeebs_MX:MX_PCB_1.00u, F.Cu at (136.3, 54.0)
- added S20: y, ScottoKeebs_MX:MX_PCB_1.00u, F.Cu at (50.3, 96.9)
- added S21: h, ScottoKeebs_MX:MX_PCB_1.00u, F.Cu at (69.3, 115.9)
- added S22: 7, ScottoKeebs_MX:MX_PCB_1.00u, F.Cu at (155.4, 54.0)
- added S23: u, ScottoKeebs_MX:MX_PCB_1.00u, F.Cu at (114.6, 122.6)
- added S24: j, ScottoKeebs_MX:MX_PCB_1.00u, F.Cu at (98.9, 135.0)
- added S25: 8, ScottoKeebs_MX:MX_PCB_1.00u, F.Cu at (174.4, 54.0)
- added S26: i, ScottoKeebs_MX:MX_PCB_1.00u, F.Cu at (30.8, 188.6)
- added S27: k, ScottoKeebs_MX:MX_PCB_1.00u, F.Cu at (100.0, 181.6)
- added S28: 9, ScottoKeebs_MX:MX_PCB_1.00u, F.Cu at (193.5, 54.0)
- added S29: o, ScottoKeebs_MX:MX_PCB_1.00u, F.Cu at (93.4, 91.1)
- added S30: l, ScottoKeebs_MX:MX_PCB_1.00u, F.Cu at (115.6, 85.1)
- added S31: 0, ScottoKeebs_MX:MX_PCB_1.00u, F.Cu at (212.5, 54.0)
- added S32: p, ScottoKeebs_MX:MX_PCB_1.00u, F.Cu at (87.1, 115.2)
- added S33: ;, ScottoKeebs_MX:MX_PCB_1.00u, F.Cu at (26.7, 118.6)
- added S37: -, ScottoKeebs_MX:MX_PCB_1.00u, F.Cu at (231.6, 54.0)
- added S38: [, ScottoKeebs_MX:MX_PCB_1.00u, F.Cu at (52.5, 157.5)
- added S39: ', ScottoKeebs_MX:MX_PCB_1.00u, F.Cu at (115.6, 181.6)
- added S40: =, ScottoKeebs_MX:MX_PCB_1.00u, F.Cu at (250.6, 54.0)
- added S41: ], ScottoKeebs_MX:MX_PCB_1.00u, F.Cu at (150.9, 82.6)
- added S42: enter, ScottoKeebs_MX:MX_PCB_1.00u, F.Cu at (130.7, 75.6)
- added S43: shift, ScottoKeebs_MX:MX_PCB_1.00u, F.Cu at (131.1, 103.9)
- added S44: ctrl, ScottoKeebs_MX:MX_PCB_1.00u, F.Cu at (47.4, 134.8)
- added S45: z, ScottoKeebs_MX:MX_PCB_1.00u, F.Cu at (189.0, 135.0)
- added S46: windows, ScottoKeebs_MX:MX_PCB_1.00u, F.Cu at (131.1, 150.5)
- added S47: x, ScottoKeebs_MX:MX_PCB_1.00u, F.Cu at (146.4, 162.7)
- added S48: alt, ScottoKeebs_MX:MX_PCB_1.00u, F.Cu at (131.1, 181.6)
- added S49: c, ScottoKeebs_MX:MX_PCB_1.00u, F.Cu at (107.8, 25.4)
- added S50: space, ScottoKeebs_MX:MX_PCB_1.00u, F.Cu at (146.7, 72.8)
- added S51: v, ScottoKeebs_MX:MX_PCB_1.00u, F.Cu at (236.7, 82.6)
- added S52: altright, ScottoKeebs_MX:MX_PCB_1.00u, F.Cu at (146.7, 103.9)
- added S53: b, ScottoKeebs_MX:MX_PCB_1.00u, F.Cu at (127.6, 131.6)
- added S54: windowsright, ScottoKeebs_MX:MX_PCB_1.00u, F.Cu at (146.7, 135.0)
- added S55: n, ScottoKeebs_MX:MX_PCB_1.00u, F.Cu at (96.8, 159.5)
- added S56: page, ScottoKeebs_MX:MX_PCB_1.00u, F.Cu at (164.9, 166.1)
- added S57: m, ScottoKeebs_MX:MX_PCB_1.00u, F.Cu at (146.7, 181.6)
- added S58: ctrlright, ScottoKeebs_MX:MX_PCB_1.00u, F.Cu at (88.7, 25.4)
- added S59: ,, ScottoKeebs_MX:MX_PCB_1.00u, F.Cu at (162.2, 72.8)
- added S61: ., ScottoKeebs_MX:MX_PCB_1.00u, F.Cu at (186.5, 87.6)
- added S63: /, ScottoKeebs_MX:MX_PCB_1.00u, F.Cu at (162.2, 103.9)
- added S67: shiftright, ScottoKeebs_MX:MX_PCB_1.00u, F.Cu at (185.7, 111.9)
- added S71: backspace, ScottoKeebs_MX:MX_PCB_1.00u, F.Cu at (278.2, 54.0)
- added S72: \, ScottoKeebs_MX:MX_PCB_1.00u, F.Cu at (173.2, 146.7)
- D1, D2, D3, D4, D5, D6, D7, D8, D9: moved to F.Cu
- S1: value Keyswitch -> esc
- S2: value Keyswitch -> 1
- S3: value Keyswitch -> 2
- S4: value Keyswitch -> tab
- S5: value Keyswitch -> q
- S6: value Keyswitch -> w
- S7: value Keyswitch -> caps
- S8: value Keyswitch -> a
- S9: value Keyswitch -> s
- moved S8 133.3 mm to (31.6, 166.1)
- moved S9 124.3 mm to (68.9, 181.6)
- moved S7 115.7 mm to (24.3, 147.0)
- moved S1 115.4 mm to (22.0, 54.0)
- moved S2 115.4 mm to (41.1, 54.0)
- moved S3 115.4 mm to (60.1, 54.0)
- moved S4 110.7 mm to (26.8, 73.0)
- moved S6 106.0 mm to (69.7, 73.0)
- moved S5 106.0 mm to (50.6, 73.0)
- moved U1 89.3 mm to (275.4, 141.0)
- moved D1 72.8 mm to (208.1, 114.9), turned to 0 degrees
- moved D4 69.0 mm to (208.1, 125.5), turned to 0 degrees
- moved D7 66.1 mm to (208.1, 136.2), turned to 0 degrees
- moved D2 59.3 mm to (208.1, 118.4), turned to 0 degrees
- moved D5 54.1 mm to (208.1, 129.1), turned to 0 degrees
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Connections:
- U1 pad 10: unconnected-(U1-GPIO7-Pad10) -> col2
- U1 pad 11: unconnected-(U1-GPIO8-Pad11) -> col3
- U1 pad 12: unconnected-(U1-GPIO9-Pad12) -> col4
- U1 pad 14: unconnected-(U1-GPIO10-Pad14) -> col5
- U1 pad 15: unconnected-(U1-GPIO11-Pad15) -> col6
- U1 pad 16: unconnected-(U1-GPIO12-Pad16) -> col7
- U1 pad 17: unconnected-(U1-GPIO13-Pad17) -> col8
- U1 pad 19: unconnected-(U1-GPIO14-Pad19) -> col9
- U1 pad 20: unconnected-(U1-GPIO15-Pad20) -> col10
- U1 pad 26: unconnected-(U1-GPIO20-Pad26) -> col13
- U1 pad 27: unconnected-(U1-GPIO21-Pad27) -> col12
- U1 pad 29: unconnected-(U1-GPIO22-Pad29) -> col11
- U1 pad 5: col0 -> row3
- U1 pad 6: col1 -> row4
- U1 pad 7: col2 -> col0
- U1 pad 9: unconnected-(U1-GPIO6-Pad9) -> col1
Routing:
- net col0: track 103.1 -> 0.00 mm
- net col1: track 84.1 -> 0.00 mm
- net row2: track 80.7 -> 0.00 mm
- net col2: track 68.4 -> 0.00 mm
- net row1: track 66.9 -> 0.00 mm
- net row0: track 50.2 -> 0.00 mm
- net Net-(D3-A): track 7.12 -> 0.00 mm
- net Net-(D9-A): track 7.12 -> 0.00 mm
- net Net-(D6-A): track 7.12 -> 0.00 mm
- net Net-(D2-A): track 7.12 -> 0.00 mm
- net Net-(D1-A): track 7.12 -> 0.00 mm
- net Net-(D8-A): track 7.12 -> 0.00 mm
- net Net-(D7-A): track 7.12 -> 0.00 mm
- net Net-(D5-A): track 7.12 -> 0.00 mm
- net Net-(D4-A): track 7.12 -> 0.00 mm
- removed copper zone on B.Cu, net (none)
- removed copper zone on F.Cu, net (none)
Other:
- board outline removed

Commit message: New Wires
Parts:
- added C23: 10uF, Capacitor_SMD:C_0805_2012Metric_Pad1.18x1.45mm_HandSolder, F.Cu at (127.0, 113.5)
- added C24: 10uF, Capacitor_SMD:C_0805_2012Metric_Pad1.18x1.45mm_HandSolder, F.Cu at (131.6, 107.7)
- added C25: 100nF, Capacitor_SMD:C_0805_2012Metric_Pad1.18x1.45mm_HandSolder, F.Cu at (125.6, 107.7)
- added D34: SD1206T020S1R0, Diode_SMD:D_1206_3216Metric_Pad1.42x1.75mm_HandSolder, F.Cu at (106.3, 114.7)
- added J1: USB_C_Receptacle_USB2.0, Connector_USB:USB_C_Receptacle_HRO_TYPE-C-31-M-12, F.Cu at (97.0, 109.9)
- added J2: USB_C_Receptacle_USB2.0, Connector_USB:USB_C_Receptacle_HRO_TYPE-C-31-M-12, F.Cu at (153.0, 109.9)
- added J4: USB_C_Receptacle_USB2.0, Connector_USB:USB_C_Receptacle_HRO_TYPE-C-31-M-12, F.Cu at (164.9, 109.9)
- added J5: USB_C_Receptacle_USB2.0, Connector_USB:USB_C_Receptacle_HRO_TYPE-C-31-M-12, F.Cu at (176.8, 109.9)
- added J6: PGA2040, footprints:PGA2040_PTH_NO_SLOT, B.Cu at (173.2, 201.2)
- added R1: 5.1K, Resistor_SMD:R_0805_2012Metric_Pad1.20x1.40mm_HandSolder, F.Cu at (105.4, 110.9)
- added R14: 56K, Resistor_SMD:R_0805_2012Metric_Pad1.20x1.40mm_HandSolder, F.Cu at (132.8, 114.3)
- added R15: 56K, Resistor_SMD:R_0805_2012Metric_Pad1.20x1.40mm_HandSolder, F.Cu at (138.3, 109.9)
- added R16: 56K, Resistor_SMD:R_0805_2012Metric_Pad1.20x1.40mm_HandSolder, F.Cu at (136.3, 114.5)
- added R17: 56K, Resistor_SMD:R_0805_2012Metric_Pad1.20x1.40mm_HandSolder, F.Cu at (139.9, 114.7)
- added R18: 56K, Resistor_SMD:R_0805_2012Metric_Pad1.20x1.40mm_HandSolder, F.Cu at (184.0, 113.7)
- added R19: 56K, Resistor_SMD:R_0805_2012Metric_Pad1.20x1.40mm_HandSolder, F.Cu at (143.5, 114.5)
- added R2: 5.1K, Resistor_SMD:R_0805_2012Metric_Pad1.20x1.40mm_HandSolder, F.Cu at (89.9, 113.7)
- added REF**: Stabilizer_MX_3.00u, ScottoKeebs_Stabilizer:Stabilizer_MX_3.00u, F.Cu at (341.1, 182.6)
- added REF**: Stabilizer_MX_2.00u, ScottoKeebs_Stabilizer:Stabilizer_MX_2.00u, F.Cu at (348.3, 163.5)
- added REF**: Stabilizer_MX_8.00u, ScottoKeebs_Stabilizer:Stabilizer_MX_8.00u, F.Cu at (214.9, 201.6)
- added REF**: Stabilizer_MX_2.00u, ScottoKeebs_Stabilizer:Stabilizer_MX_2.00u, F.Cu at (103.0, 163.5)
- added REF**: Stabilizer_MX_2.00u, ScottoKeebs_Stabilizer:Stabilizer_MX_2.00u, F.Cu at (350.6, 125.4)
- added REF**: Stabilizer_MX_2.00u, ScottoKeebs_Stabilizer:Stabilizer_MX_2.00u, F.Cu at (105.4, 182.6)
- added REF**: Stabilizer_MX_2.00u, ScottoKeebs_Stabilizer:Stabilizer_MX_2.00u, F.Cu at (103.0, 144.5)
- added SW3: RESET, Button_Switch_SMD:SW_Push_1P1T_NO_Vertical_Wuerth_434133025816, B.Cu at (187.9, 195.8)
- added SW4: BOOTSEL, Button_Switch_SMD:SW_Push_1P1T_NO_Vertical_Wuerth_434133025816, B.Cu at (187.5, 201.6)
- D1, D10, D11, D12, D13, D14, D15, D16, D17, D18, D19, D2, D20, D21, D22, D23, D24, D25, D26, D27, D28, D29, D3, D30, D31, D32, D33, D37, D38, D39, D4, D40, D41, D42, D43, D44, D45, D46, D47, D48, D49, D5, D50, D51, D52, D53, D54, D55, D56, D57, D58, D59, D6, D61, D63, D67, D7, D71, D72, D8, D9: moved to B.Cu
- U1: value Raspberry_Pi_Pico -> SL2.1A; footprint ScottoKeebs_MCU:Raspberry_Pi_Pico -> Package_SO:SOIC-16_4.55x10.3mm_P1.27mm
- moved S58 317.7 mm to (353.0, 201.6)
- moved S33 277.6 mm to (300.6, 163.5)
- moved S38 267.5 mm to (319.7, 144.5)
- moved S26 235.9 mm to (262.5, 144.5)
- moved S42 234.6 mm to (348.3, 163.5)
- moved S32 215.6 mm to (300.6, 144.5)
- moved S39 204.9 mm to (319.7, 163.5)
- moved S41 197.7 mm to (338.7, 144.5)
- moved S29 195.6 mm to (281.6, 144.5)
- moved S72 184.6 mm to (357.8, 144.5)
- moved S30 183.6 mm to (281.6, 163.5)
- moved S54 181.0 mm to (314.9, 201.6)
- moved S20 180.5 mm to (224.4, 144.5)
- moved S52 178.4 mm to (295.9, 201.6)
- moved S56 172.8 mm to (334.0, 201.6)
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Connections:
- U1 pad 1: row0 -> /D4-
- U1 pad 10: col2 -> /USB_D+
- U1 pad 11: col3 -> /USBC_VBUS
- U1 pad 12: col4 -> USBC_GND
- U1 pad 13: unconnected-(U1-GND-Pad13)_1 -> Net-(U1-VDD3)
- U1 pad 14: col5 -> Net-(U1-VDD18)
- U1 pad 15: col6 -> unconnected-(U1-XOUT-Pad15)
- U1 pad 16: col7 -> USBC_GND
- U1 pad 2: row1 -> /D4+
- U1 pad 3: unconnected-(U1-GND-Pad3) -> /D3-
- U1 pad 4: row2 -> /D3+
- U1 pad 5: row3 -> /D2-
- U1 pad 6: row4 -> /D2+
- U1 pad 7: col0 -> /D1-
- U1 pad 8: unconnected-(U1-GND-Pad8)_1 -> /D1+
- U1 pad 9: col1 -> /USB_D-
Routing:
- net col13: track 0.00 -> 494.4 mm
- net col10: track 0.00 -> 460.2 mm
- net col6: track 0.00 -> 366.1 mm, vias 0 -> 1
- net col11: track 0.00 -> 336.4 mm
- net col5: track 0.00 -> 322.3 mm, vias 0 -> 1
- net row4: track 0.00 -> 275.1 mm
- net col9: track 0.00 -> 273.4 mm
- net row0: track 0.00 -> 262.8 mm
- net row1: track 0.00 -> 262.6 mm
- net row2: track 0.00 -> 260.5 mm
- net row3: track 0.00 -> 243.1 mm
- net col0: track 0.00 -> 222.6 mm
- net col1: track 0.00 -> 217.6 mm
- net USBC_GND: track 0.00 -> 210.3 mm, vias 0 -> 1
- net col4: track 0.00 -> 182.0 mm
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Other:
- board outline added: 284.6 x 108.9 mm
