File: pcb/pcb.kicad_sch (KiCad schematic)
At the start: 123 parts, among them U1 Raspberry_Pi_Pico

Commit message: New Wires
Parts:
- removed U1: Raspberry_Pi_Pico, ScottoKeebs_MCU:Raspberry_Pi_Pico, symbol ScottoKeebs:MCU_Raspberry_Pi_Pico
- added C23, C24: 10uF, Capacitor_SMD:C_0805_2012Metric_Pad1.18x1.45mm_HandSolder, symbol Device:C_Small
- added C25: 100nF, Capacitor_SMD:C_0805_2012Metric_Pad1.18x1.45mm_HandSolder, symbol Device:C_Small
- added D34: SD1206T020S1R0, Diode_SMD:D_1206_3216Metric_Pad1.42x1.75mm_HandSolder, symbol Device:D_Small
- added J1, J2, J4, J5: USB_C_Receptacle_USB2.0, Connector_USB:USB_C_Receptacle_HRO_TYPE-C-31-M-12, symbol Connector:USB_C_Receptacle_USB2.0
- added J6: PGA2040, footprints:PGA2040_PTH_NO_SLOT, symbol PGA2040:PGA2040
- added R1, R2: 5.1K, Resistor_SMD:R_0805_2012Metric_Pad1.20x1.40mm_HandSolder, symbol Device:R_Small
- added R14, R15, R16, R17, R18, R19: 56K, Resistor_SMD:R_0805_2012Metric_Pad1.20x1.40mm_HandSolder, symbol Device:R_Small
- added SW3: RESET, Button_Switch_SMD:SW_Push_1P1T_NO_Vertical_Wuerth_434133025816, symbol Switch:SW_Push
- added SW4: BOOTSEL, Button_Switch_SMD:SW_Push_1P1T_NO_Vertical_Wuerth_434133025816, symbol Switch:SW_Push
- added U1: SL2.1A, Package_SO:SOIC-16_4.55x10.3mm_P1.27mm, symbol SL2.1A:SL2.1A
Connections:
- net col0: now also J6.E1 (GPIO5)
- net col1: now also J6.E2 (GPIO6)
- net col10: now also J6.H5 (GPIO15)
- net col11: now also J6.G5 (GPIO16)
- net col12: now also J6.H6 (GPIO17)
- net col13: now also J6.G6 (GPIO18)
- net col2: now also J6.F1 (GPIO7)
- net col3: now also J6.F2 (GPIO8)
- net col4: now also J6.G1 (GPIO9)
- net col5: now also J6.H2 (GPIO10)
- net col6: now also J6.H3 (GPIO11)
- net col7: now also J6.G3 (GPIO12)
- net col8: now also J6.H4 (GPIO13)
- net col9: now also J6.G4 (GPIO14)
- net row0: now also J6.B1 (GPIO0)
- net row1: now also J6.C1 (GPIO1)
- net row2: now also J6.C2 (GPIO2)
- net row3: now also J6.D1 (GPIO3)
- net row4: now also J6.D2 (GPIO4)
- new net: J6.A7 (BOOTSEL), SW4.2
- new net: J6.A4 (RUN), SW3.2
- new net: J2.B5 (CC2), R15.1
- new net: J4.A5 (CC1), R16.2
- new net: J2.A5 (CC1), R14.2
- new net: J5.A5 (CC1), R18.2
- new net: J1.A5 (CC1), R1.2
- new net: J1.B5 (CC2), R2.1
- new net: J5.B5 (CC2), R19.1
- new net: D34.2 (A), J1.A4 (VBUS), J1.A9 (VBUS), J1.B4 (VBUS), J1.B9 (VBUS)
- new net: C23.1, U1.13 (VDD3)
- new net: C24.2, U1.14 (VDD18)
- new net: J4.B5 (CC2), R17.1
- new net D1+: J2.A6 (D+), J2.B6 (D+), U1.8 (DP1)
- new net D1-: J2.A7 (D-), J2.B7 (D-), U1.7 (DM1)
- new net D2+: J4.A6 (D+), J4.B6 (D+), U1.6 (DP2)
- new net D2-: J4.A7 (D-), J4.B7 (D-), U1.5 (DM2)
- new net D3+: J5.A6 (D+), J5.B6 (D+), U1.4 (DP3)
- new net D3-: J5.A7 (D-), J5.B7 (D-), U1.3 (DM3)
- new net D4+: J6.A6 (USB_DM), U1.2 (DP4)
- new net D4-: J6.A5 (USB_DP), U1.1 (DM4)
- new net USBC_GND: C23.2, C24.1, C25.1, J1.A1 (GND), J1.A12 (GND), J1.B1 (GND), J1.B12 (GND), J1.S1 (SHIELD), J2.A1 (GND), J2.A12 (GND), J2.B1 (GND), J2.B12 (GND), J2.S1 (SHIELD), J4.A1 (GND), J4.A12 (GND), J4.B1 (GND), J4.B12 (GND), J4.S1 (SHIELD), J5.A1 (GND), J5.A12 (GND), J5.B1 (GND), J5.B12 (GND), J5.S1 (SHIELD), J6.A1 (GND), J6.A8 (GND), J6.B2 (GND), J6.B7 (GND), J6.G2 (GND), J6.G7 (GND), J6.H1 (GND), J6.H8 (GND), R1.1, R2.2, SW3.1, SW4.1, U1.12 (GND), U1.16 (XIN)
- new net USBC_VBUS: C25.2, D34.1 (K), J2.A4 (VBUS), J2.A9 (VBUS), J2.B4 (VBUS), J2.B9 (VBUS), J4.A4 (VBUS), J4.A9 (VBUS), J4.B4 (VBUS), J4.B9 (VBUS), J5.A4 (VBUS), J5.A9 (VBUS), J5.B4 (VBUS), J5.B9 (VBUS), J6.A2 (VBUS), R14.1, R15.2, R16.1, R17.2, R18.1, R19.2, U1.11 (VCC5V)
- new net USB_D+: J1.A6 (D+), J1.B6 (D+), U1.10 (UDP)
- new net USB_D-: J1.A7 (D-), J1.B7 (D-), U1.9 (UDM)
Other:
- note added: "Default USB Power 500mA @ 5V"
- note added: "Switches"
- note added: "USB2 Type-C Receptacle IN"
- note added: "USBC Extender"
- moved on the sheet: D1, D10, D11, D12, D13, D14, D15, D16, D17, D18, D19, D2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
